File: board/RISKYX68000.kicad_pcb (KiCad board)
At the start: 4 copper layers, 36.6 x 39.6 mm, 32 parts, among them J1 DE9_Plug, J2 Conn_01x02, J3 USB_1, J4 Conn_01x02, J5 Conn_01x02, J6 Conn_01x02, J7 Conn_01x04, U1 CH32V203C8T6, U2 LM1117MP-3.3

Commit message: First PCB order
Routing:
- net GND: track 18.5 -> 19.4 mm
Other:
- board text added: "1"
- board text added: "2"
- board text added: "3"
- board text added: "4"
- board text added: "5"
- board text removed: "D1"
- board text removed: "D2"
- board text removed: "D3"
- board text removed: "D4"
- board text removed: "D5"
Changed lines of the file:
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@@
 			(at 0 10 0)
 			(layer "F.Fab")
+			(hide yes)
 			(effects
 				(font
@@
 		(tags "LQFP QFP")
 		(property "Reference" "U1"
-			(at 0 -5.85 0)
+			(at 0.435 -5.8525 0)
 			(layer "F.SilkS")
 			(effects
@@
 		(tags "SOT-89-3")
 		(property "Reference" "U2"
-			(at -3.6274 1.524 90)
+			(at 0.0725 -4.37 90)
 			(layer "F.SilkS")
+			(hide yes)
 			(effects
 				(font
@@
 		(attr smd)
 		(fp_line
-			(start -1.36 2.36)
-			(end -1.36 2.13)
-			(stroke
-				(width 0.12)
-				(type solid)
-			)
-			(layer "F.SilkS")
-		)
-		(fp_line
 			(start 1.36 2.36)
 			(end -1.36 2.36)
@@
 		)
 		(fp_line
-			(start -2.5 -2.13)
-			(end -1.36 -2.13)
-			(stroke
-				(width 0.12)
-				(type solid)
-			)
-			(layer "F.SilkS")
-		)
-		(fp_line
-			(start -1.36 -2.36)
-			(end -1.36 -2.13)
-			(stroke
-				(width 0.12)
-				(type solid)
-			)
-			(layer "F.SilkS")
-		)
-		(fp_line
 			(start -1.36 -2.36)
 			(end 1.36 -2.36)
@@
 		(tags "capacitor handsolder")
 		(property "Reference" "C2"
-			(at -0.0254 -1.3208 0)
+			(at 1.5528 1.156 0)
 			(layer "B.SilkS")
+			(hide yes)
 			(effects
 				(font
@@
 		(attr smd)
 		(fp_line
-			(start -0.146267 -0.51)
-			(end 0.146267 -0.51)
-			(stroke
-				(width 0.12)
-				(type solid)
-			)
-			(layer "B.SilkS")
-		)
-		(fp_line
-			(start -0.146267 0.51)
-			(end 0.146267 0.51)
-			(stroke
-				(width 0.12)
-				(type solid)
-			)
-			(layer "B.SilkS")
-		)
-		(fp_line
 			(start -1.65 -0.73)
 			(end -1.65 0.73)
@@
 			(at 0.1078 -1.7122 270)
 			(layer "B.SilkS")
+			(hide yes)
 			(effects
 				(font
@@
 		(layer "Edge.Cuts")
 	)
-	(gr_text "D3\n"
-		(at 119.475 88.125 0)
+	(gr_text "3"
+		(at 119.9 88.25 0)
 		(layer "F.SilkS")
 		(effects
@@
 		)
 	)
-	(gr_text "D5\n\n"
-		(at 119.5 94.95 0)
+	(gr_text "5"
+		(at 119.875 92.575 0)
 		(layer "F.SilkS")
 		(effects
@@
 		)
 	)
-	(gr_text "D1"
-		(at 119.5 83.9 0)
+	(gr_text "1"
+		(at 119.85 83.95 0)
 		(layer "F.SilkS")
 		(effects
@@
 		)
 	)
-	(gr_text "D4\n"
-		(at 119.525 90.4 0)
+	(gr_text "4"
+		(at 119.9 90.5 0)
 		(layer "F.SilkS")
 		(effects
@@
 		)
 	)
-	(gr_text "D2\n"
-		(at 119.525 86.025 0)
+	(gr_text "2"
+		(at 119.85 86.05 0)
 		(layer "F.SilkS")
 		(effects
@@
 	)
 	(segment
-		(start 125.596121 93.916221)
-		(end 125.5861 93.9062)
-		(width 0.127)
-		(layer "F.Cu")
-		(net 1)
-	)
-	(segment
 		(start 126.9986 90.0146)
 		(end 126.9986 90.2364)
@@
 	)
 	(segment
-		(start 126.9986 88.4937)
-		(end 126.9986 90.0146)
-		(width 0.2)
+		(start 127.191279 93.916221)
+		(end 125.596121 93.916221)
+		(width 0.127)
 		(layer "F.Cu")
 		(net 1)
 	)
 	(segment
-		(start 126.8902 89.9062)
+		(start 126.9986 88.4937)
 		(end 126.9986 90.0146)
 		(width 0.2)
@@
 	)
 	(segment
-		(start 126.530218 93.916221)
-		(end 125.596121 93.916221)
+		(start 125.596121 93.916221)
+		(end 125.5861 93.9062)
 		(width 0.127)
 		(layer "F.Cu")
@@
 	)
 	(segment
+		(start 126.8902 89.9062)
+		(end 126.9986 90.0146)
+		(width 0.2)
+		(layer "F.Cu")
+		(net 1)
+	)
+	(segment
 		(start 126.9986 90.2364)
 		(end 127.107 90.3448)
@@
 	)
 	(segment
+		(start 127.4372 93.6703)
+		(end 127.191279 93.916221)
+		(width 0.127)
+		(layer "F.Cu")
+		(net 1)
+	)
+	(segment
 		(start 132.4664 95.8312)
 		(end 132.4664 96.7865)
@@
 	)
 	(via
-		(at 126.530218 93.916221)
+		(at 127.4372 93.6703)
 		(size 0.6)
 		(drill 0.3)
@@
 	)
 	(segment
-		(start 126.530218 94.264918)
-		(end 126.530218 93.916221)
-		(width 0.127)
-		(layer "B.Cu")
-		(net 1)
-	)
-	(segment
-		(start 127.5134 95.2481)
-		(end 126.530218 94.264918)
-		(width 0.127)
-		(layer "B.Cu")
-		(net 1)
-	)
-	(segment
 		(start 122.5834 98.6934)
 		(end 122.63 98.74)
@@
 	)
 	(segment
-		(start 126.776139 93.6703)
-		(end 126.530218 93.916221)
-		(width 0.127)
-		(layer "B.Cu")
-		(net 1)
-	)
-	(segment
 		(start 132.4399 95.8047)
 		(end 132.4664 95.8312)
@@
 	)
 	(segment
+		(start 127.4372 95.1719)
+		(end 127.5134 95.2481)
+		(width 0.127)
+		(layer "B.Cu")
+		(net 1)
+	)
+	(segment
 		(start 126.1219 95.2481)
 		(end 122.63 98.74)
@@
 	(segment
 		(start 127.4372 93.6703)
-		(end 126.776139 93.6703)
+		(end 127.4372 95.1719)
 		(width 0.127)
 		(layer "B.Cu")
@@
 	)
 	(segment
+		(start 131.99 98.09)
+		(end 131.99 96.815)
+		(width 0.127)
+		(layer "F.Cu")
+		(net 2)
+	)
+	(segment
+		(start 124.3 93.025)
+		(end 124.3 93.064543)
+		(width 0.127)
+		(layer "F.Cu")
+		(net 2)
+	)
+	(segment
 		(start 133.9025 90.4025)
 		(end 134.8975 90.4025)
@@
 	)
 	(segment
-		(start 131.98 98.1)
-		(end 131.99 98.09)
+		(start 124.3 93.064543)
+		(end 124.637957 93.4025)
 		(width 0.127)
 		(layer "F.Cu")
@@
 	)
 	(segment
+		(start 124.637957 93.4025)
+		(end 125.5775 93.4025)
+		(width 0.127)
+		(layer "F.Cu")
+		(net 2)
+	)
+	(segment
 		(start 130.49 95.11)
 		(end 130.7 94.9)
@@
 	)
 	(segment
-		(start 127.49 87.01)
-		(end 127.5 87)
+		(start 124.25 92.975)
+		(end 124.3 93.025)
 		(width 0.127)
 		(layer "F.Cu")
@@
 	)
 	(segment
-		(start 124.637957 93.4025)
-		(end 124.61862 93.383163)
+		(start 127.49 87.01)
+		(end 127.5 87)
 		(width 0.127)
 		(layer "F.Cu")
@@
 	)
 	(segment
-		(start 131.99 98.09)
-		(end 131.99 96.815)
+		(start 132.1 98.2)
+		(end 131.99 98.09)
 		(width 0.127)
 		(layer "F.Cu")
@@
 	)
 	(segment
-		(start 125.5775 93.4025)
-		(end 124.637957 93.4025)
+		(start 132.375 98.2)
+		(end 132.1 98.2)
 		(width 0.127)
 		(layer "F.Cu")
@@
 	)
 	(via
-		(at 131.98 98.1)
+		(at 132.375 98.2)
 		(size 0.6)
 		(drill 0.3)
@@
 	)
 	(via
-		(at 124.61862 93.383163)
+		(at 124.25 92.975)
 		(size 0.6)
 		(drill 0.3)
@@
 	)
 	(segment
-		(start 126.566051 92.941667)
+		(start 127.4372 91.8453)
+		(end 126.340833 92.941667)
+		(width 0.127)
+		(layer "F.Cu")
+		(net 4)
+	)
+	(segment
+		(start 126.340833 92.941667)
 		(end 125.621567 92.941667)
 		(width 0.127)
@@
 	)
 	(via
-		(at 126.566051 92.941667)
+		(at 127.4372 91.8453)
 		(size 0.6)
 		(drill 0.3)
@@
 	)
 	(segment
-		(start 127.4372 92.070518)
-		(end 126.566051 92.941667)
-		(width 0.127)
-		(layer "B.Cu")
-		(net 4)
-	)
-	(segment
-		(start 127.4372 91.8453)
-		(end 127.4372 92.070518)
-		(width 0.127)
-		(layer "B.Cu")
-		(net 4)
-	)
-	(segment
 		(start 133.675 82.05)
 		(end 134.95 80.775)
@@
 	)
 	(segment
-		(start 131.49 96.815)
-		(end 131.49 97.718184)
+		(start 131.492457 98.307543)
+		(end 131.492457 97.720641)
 		(width 0.127)
 		(layer "F.Cu")
@@
 	(segment
 		(start 131.49 97.718184)
-		(end 131.271604 97.93658)
+		(end 131.49 96.815)
+		(width 0.127)
+		(layer "F.Cu")
+		(net 41)
+	)
+	(segment
+		(start 131.492457 97.720641)
+		(end 131.49 97.718184)
 		(width 0.127)
 		(layer "F.Cu")
@@
 	)
 	(via
-		(at 131.271604 97.93658)
+		(at 131.492457 98.307543)
 		(size 0.6)
 		(drill 0.3)
@@
 	)
 	(segment
-		(start 131.271604 98.08669)
-		(end 131.271604 97.93658)
-		(width 0.127)
-		(layer "B.Cu")
-		(net 41)
-	)
-	(segment
 		(start 143.2255 98.9755)
-		(end 132.160414 98.9755)
+		(end 144.55 100.3)
 		(width 0.127)
 		(layer "B.Cu")
@@
 	)
 	(segment
-		(start 144.55 100.3)
+		(start 132.160414 98.9755)
 		(end 143.2255 98.9755)
 		(width 0.127)
@@
 	)
 	(segment
-		(start 132.160414 98.9755)
-		(end 131.271604 98.08669)
+		(start 131.492457 98.307543)
+		(end 132.160414 98.9755)
 		(width 0.127)
 		(layer "B.Cu")
